File: device/impact_v1/impact_v1.kicad_sch (KiCad schematic)
At the start: 21 parts, among them J1 Conn_01x02_Female, U1 MIC5200-3.3YM, U2 MPU-6050, U3 ADXL375, U4 ESP32-WROOM-32D

Commit message: Routing
Parts:
- removed J1: Conn_01x02_Female, Connector_Wire:SolderWire-1sqmm_1x02_P5.4mm_D1.4mm_OD2.7mm, symbol Connector:Conn_01x02_Female
- added J1, J2: Conn_01x01_Male, TestPoint:TestPoint_Pad_D4.0mm, symbol Connector:Conn_01x01_Male
- C2: footprint (none) -> Capacitor_SMD:C_1206_3216Metric_Pad1.33x1.80mm_HandSolder
- D1: renamed from D?; footprint (none) -> Diode_SMD:D_0402_1005Metric_Pad0.77x0.64mm_HandSolder
- U1: footprint Resistor_SMD:R_0603_1608Metric_Pad0.98x0.95mm_HandSolder -> Voltage_Regulator_Linear:MIC5200-3.3YM
Connections:
- net +BATT: now also J1.1 (Pin_1)
- net GND: now also U4.1 (GND), U4.15 (GND), U4.38 (GND), U4.39 (GND), J2.1 (Pin_1)
- net VDD: no longer U2.12 (INT), U4.29 (IO5)
- new net: U2.12 (INT), U4.29 (IO5)
Changed lines of the file:
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@@
   (junction (at 83.185 106.68) (diameter 0) (color 0 0 0 0)
   )
-  (junction (at 139.065 147.32) (diameter 0) (color 0 0 0 0)
-  )
   (wire (pts (xy 259.715 67.31) (xy 259.715 70.485))
     (stroke (width 0) (type default) (color 0 0 0 0))
@@
     (stroke (width 0) (type default) (color 0 0 0 0))
   )
+  (wire (pts (xy 172.72 158.115) (xy 262.255 158.115))
+    (stroke (width 0) (type default) (color 0 0 0 0))
+  )
   (wire (pts (xy 99.695 91.44) (xy 98.425 91.44))
     (stroke (width 0) (type default) (color 0 0 0 0))
@@
     (stroke (width 0) (type default) (color 0 0 0 0))
   )
+  (wire (pts (xy 172.72 166.37) (xy 172.72 158.115))
+    (stroke (width 0) (type default) (color 0 0 0 0))
+  )
   (wire (pts (xy 262.255 95.25) (xy 252.73 95.25))
     (stroke (width 0) (type default) (color 0 0 0 0))
@@
     (stroke (width 0) (type default) (color 0 0 0 0))
   )
-  (wire (pts (xy 139.065 147.32) (xy 262.255 147.32))
-    (stroke (width 0) (type default) (color 0 0 0 0))
-  )
   (wire (pts (xy 152.4 36.83) (xy 160.02 36.83))
     (stroke (width 0) (type default) (color 0 0 0 0))
@@
     (stroke (width 0) (type default) (color 0 0 0 0))
   )
-  (wire (pts (xy 127.635 147.32) (xy 139.065 147.32))
-    (stroke (width 0) (type default) (color 0 0 0 0))
-  )
   (wire (pts (xy 264.795 60.325) (xy 269.875 60.325))
     (stroke (width 0) (type default) (color 0 0 0 0))
@@
     (stroke (width 0) (type default) (color 0 0 0 0))
   )
+  (wire (pts (xy 127.635 147.32) (xy 127.635 166.37))
+    (stroke (width 0) (type default) (color 0 0 0 0))
+  )
   (wire (pts (xy 131.445 140.97) (xy 131.445 142.24))
     (stroke (width 0) (type default) (color 0 0 0 0))
   )
+  (wire (pts (xy 127.635 166.37) (xy 172.72 166.37))
+    (stroke (width 0) (type default) (color 0 0 0 0))
+  )
   (wire (pts (xy 96.52 34.29) (xy 83.82 34.29))
     (stroke (width 0) (type default) (color 0 0 0 0))
@@
     (stroke (width 0) (type default) (color 0 0 0 0))
   )
-  (wire (pts (xy 262.255 147.32) (xy 262.255 95.25))
+  (wire (pts (xy 262.255 95.25) (xy 262.255 158.115))
     (stroke (width 0) (type default) (color 0 0 0 0))
   )
@@
   (symbol (lib_id "Device:D_Schottky") (at 75.184 50.8 180) (unit 1)
     (in_bom yes) (on_board yes) (fields_autoplaced)
-    (property "Reference" "D?" (id 0) (at 75.5015 44.45 0))
+    (property "Reference" "D1" (id 0) (at 75.5015 44.45 0))
     (property "Value" "D_Schottky" (id 1) (at 75.5015 46.99 0))
-    (property "Footprint" "" (id 2) (at 75.184 50.8 0)
+    (property "Footprint" "Diode_SMD:D_0402_1005Metric_Pad0.77x0.64mm_HandSolder" (id 2) (at 75.184 50.8 0)
       (effects (font (size 1.27 1.27)) hide)
     )
@@
     (pin "1")
     (pin "2")
+  )
+  (symbol (lib_id "Connector:Conn_01x01_Male") (at 25.4 20.32 270) (unit 1)
+    (in_bom yes) (on_board yes)
+    (property "Reference" "J1" (id 0) (at 26.035 24.765 90)
+      (effects (font (size 1.27 1.27)) (justify left))
+    )
+    (property "Value" "Conn_01x01_Male" (id 1) (at 21.59 19.05 90)
+      (effects (font (size 1.27 1.27)) (justify left))
+    )
+    (property "Footprint" "TestPoint:TestPoint_Pad_D4.0mm" (id 2) (at 25.4 20.32 0)
+      (effects (font (size 1.27 1.27)) hide)
+    )
+    (property "Datasheet" "~" (id 3) (at 25.4 20.32 0)
+      (effects (font (size 1.27 1.27)) hide)
+    )
+    (pin "1")
   )
   (symbol (lib_id "power:+BATT") (at 25.4 25.4 180) (unit 1)
@@
     (pin "2")
   )
-  (symbol (lib_id "power:GND") (at 27.94 25.4 90) (unit 1)
-    (in_bom yes) (on_board yes) (fields_autoplaced)
-    (property "Reference" "#PWR0110" (id 0) (at 34.29 25.4 0)
-      (effects (font (size 1.27 1.27)) hide)
-    )
-    (property "Value" "GND" (id 1) (at 31.75 25.3999 90)
-      (effects (font (size 1.27 1.27)) (justify right))
-    )
-    (property "Footprint" "" (id 2) (at 27.94 25.4 0)
-      (effects (font (size 1.27 1.27)) hide)
-    )
-    (property "Datasheet" "" (id 3) (at 27.94 25.4 0)
+  (symbol (lib_id "power:GND") (at 45.085 25.4 0) (unit 1)
+    (in_bom yes) (on_board yes) (fields_autoplaced)
+    (property "Reference" "#PWR0110" (id 0) (at 45.085 31.75 0)
+      (effects (font (size 1.27 1.27)) hide)
+    )
+    (property "Value" "GND" (id 1) (at 45.085 30.48 0))
+    (property "Footprint" "" (id 2) (at 45.085 25.4 0)
+      (effects (font (size 1.27 1.27)) hide)
+    )
+    (property "Datasheet" "" (id 3) (at 45.085 25.4 0)
       (effects (font (size 1.27 1.27)) hide)
     )
@@
       (effects (font (size 1.524 1.524)))
     )
-    (property "Footprint" "Resistor_SMD:R_0603_1608Metric_Pad0.98x0.95mm_HandSolder" (id 2) (at 124.46 25.654 0)
+    (property "Footprint" "Voltage_Regulator_Linear:MIC5200-3.3YM" (id 2) (at 124.46 25.654 0)
       (effects (font (size 1.524 1.524)) hide)
     )
@@
     (pin "9")
   )
+  (symbol (lib_id "Connector:Conn_01x01_Male") (at 45.085 20.32 270) (unit 1)
+    (in_bom yes) (on_board yes)
+    (property "Reference" "J2" (id 0) (at 42.545 25.4 90)
+      (effects (font (size 1.27 1.27)) (justify left))
+    )
+    (property "Value" "Conn_01x01_Male" (id 1) (at 27.305 21.59 90)
+      (effects (font (size 1.27 1.27)) (justify left))
+    )
+    (property "Footprint" "TestPoint:TestPoint_Pad_D4.0mm" (id 2) (at 45.085 20.32 0)
+      (effects (font (size 1.27 1.27)) hide)
+    )
+    (property "Datasheet" "~" (id 3) (at 45.085 20.32 0)
+      (effects (font (size 1.27 1.27)) hide)
+    )
+    (pin "1")
+  )
   (symbol (lib_id "power:GND") (at 163.83 53.34 0) (unit 1)
     (in_bom yes) (on_board yes) (fields_autoplaced)
@@
       (effects (font (size 1.27 1.27)) (justify left))
     )
-    (property "Footprint" "" (id 2) (at 84.1502 106.68 0)
+    (property "Footprint" "Capacitor_SMD:C_1206_3216Metric_Pad1.33x1.80mm_HandSolder" (id 2) (at 84.1502 106.68 0)
       (effects (font (size 1.27 1.27)) hide)
     )
@@
     (pin "2")
   )
+  (symbol (lib_id "power:GND") (at 237.49 148.59 0) (unit 1)
+    (in_bom yes) (on_board yes) (fields_autoplaced)
+    (property "Reference" "#PWR?" (id 0) (at 237.49 154.94 0)
+      (effects (font (size 1.27 1.27)) hide)
+    )
+    (property "Value" "GND" (id 1) (at 237.49 153.67 0))
+    (property "Footprint" "" (id 2) (at 237.49 148.59 0)
+      (effects (font (size 1.27 1.27)) hide)
+    )
+    (property "Datasheet" "" (id 3) (at 237.49 148.59 0)
+      (effects (font (size 1.27 1.27)) hide)
+    )
+    (pin "1")
+  )
   (symbol (lib_id "Device:C_Small") (at 259.715 64.77 0) (unit 1)
     (in_bom yes) (on_board yes)
@@
     (pin "2")
   )
-  (symbol (lib_id "Connector:Conn_01x02_Female") (at 25.4 20.32 90) (unit 1)
-    (in_bom yes) (on_board yes) (fields_autoplaced)
-    (property "Reference" "J1" (id 0) (at 29.21 19.6849 90)
-      (effects (font (size 1.27 1.27)) (justify right))
-    )
-    (property "Value" "Conn_01x02_Female" (id 1) (at 29.21 22.2249 90)
-      (effects (font (size 1.27 1.27)) (justify right))
-    )
-    (property "Footprint" "Connector_Wire:SolderWire-1sqmm_1x02_P5.4mm_D1.4mm_OD2.7mm" (id 2) (at 25.4 20.32 0)
-      (effects (font (size 1.27 1.27)) hide)
-    )
-    (property "Datasheet" "~" (id 3) (at 25.4 20.32 0)
-      (effects (font (size 1.27 1.27)) hide)
-    )
-    (pin "1")
-    (pin "2")
-  )
   (symbol (lib_id "power:+BATT") (at 68.707 51.816 180) (unit 1)
     (in_bom yes) (on_board yes) (fields_autoplaced)
@@
       (reference "#PWR0116") (unit 1) (value "VDD") (footprint "")
     )
+    (path "/8f9431f3-fc27-41f7-bcec-faad61d8e8af"
+      (reference "#PWR?") (unit 1) (value "GND") (footprint "")
+    )
     (path "/c8b37e48-efbc-407b-86cc-d21552e503c0"
       (reference "C1") (unit 1) (value "0.01µF") (footprint "Capacitor_SMD:C_0603_1608Metric_Pad1.08x0.95mm_HandSolder")
     )
     (path "/7d055ff3-b74e-4956-8b71-3a0ca903a084"
-      (reference "C2") (unit 1) (value "10µF") (footprint "")
+      (reference "C2") (unit 1) (value "10µF") (footprint "Capacitor_SMD:C_1206_3216Metric_Pad1.33x1.80mm_HandSolder")
     )
     (path "/e660224e-d104-4e5c-999b-5cae380c0786"
@@
     )
     (path "/035ad69b-101d-4a07-9109-768fd21ef62f"
-      (reference "D?") (unit 1) (value "D_Schottky") (footprint "")
-    )
-    (path "/eb1c0288-1a6c-49e8-b97d-d84c22124b1e"
-      (reference "J1") (unit 1) (value "Conn_01x02_Female") (footprint "Connector_Wire:SolderWire-1sqmm_1x02_P5.4mm_D1.4mm_OD2.7mm")
+      (reference "D1") (unit 1) (value "D_Schottky") (footprint "Diode_SMD:D_0402_1005Metric_Pad0.77x0.64mm_HandSolder")
+    )
+    (path "/1e4bff46-8d3f-444f-a26a-b6afae30d73b"
+      (reference "J1") (unit 1) (value "Conn_01x01_Male") (footprint "TestPoint:TestPoint_Pad_D4.0mm")
+    )
+    (path "/4f1a0198-ad9a-4df1-b72e-48cd797a3682"
+      (reference "J2") (unit 1) (value "Conn_01x01_Male") (footprint "TestPoint:TestPoint_Pad_D4.0mm")
     )
     (path "/8e0c1136-87ff-4ad6-9d6e-562dfc01b098"
@@
     )
     (path "/44588560-1a8e-4995-b859-bd4c189b882b"
-      (reference "U1") (unit 1) (value "MIC5200-3.3YM") (footprint "Resistor_SMD:R_0603_1608Metric_Pad0.98x0.95mm_HandSolder")
+      (reference "U1") (unit 1) (value "MIC5200-3.3YM") (footprint "Voltage_Regulator_Linear:MIC5200-3.3YM")
     )
     (path "/3dd0cda1-793a-4812-bf87-fa5c288123be"
