File: device/impact_v1/impact_v1.kicad_pcb (KiCad board)
At the start: 2 copper layers, 32 x 27 mm, 22 parts, among them J1 Conn_01x01_Male, J2 Conn_01x01_Male, U1 MIC5200-3.3YM, U2 MPU-6050, U3 ADXL375, U4 ESP32-WROOM-32D

Commit message: End of Version 1
Routing:
- net GND: track 12.9 -> 96.4 mm, vias 0 -> 7
- net Net-(C9-Pad1): track 0.00 -> 42.5 mm, vias 0 -> 1
- net Net-(C6-Pad1): track 0.00 -> 40.6 mm, vias 0 -> 1
- net Net-(R2-Pad2): track 0.00 -> 33.6 mm, vias 0 -> 1
- net Net-(C3-Pad1): track 0.00 -> 28.6 mm
- net Net-(C1-Pad1): track 0.00 -> 21.1 mm, vias 0 -> 4
- net Net-(R1-Pad2): track 0.00 -> 15.6 mm
- net Net-(U3-Pad9): track 0.00 -> 10.7 mm
Other:
- board outline removed

Commit message: Pre Code Start
Routing:
- net GND: track 96.4 -> 92.8 mm, vias 7 -> 5
- net Net-(R2-Pad2): vias 1 -> 0
- net Net-(C1-Pad1): vias 4 -> 3
Changed lines of the file:
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@@
   (via (at 156.464 99.06) (size 0.8) (drill 0.4) (layers "F.Cu" "B.Cu") (net 1))
   (via (at 158.63931 99.71131) (size 0.8) (drill 0.4) (layers "F.Cu" "B.Cu") (net 1))
-  (via (at 155.705718 92.792209) (size 0.8) (drill 0.4) (layers "F.Cu" "B.Cu") (net 1))
   (via (at 160.994301 92.491709) (size 0.8) (drill 0.4) (layers "F.Cu" "B.Cu") (net 1))
   (segment (start 157.988 99.06) (end 158.63931 99.71131) (width 0.25) (layer "B.Cu") (net 1))
@@
   (segment (start 160.875401 83.164999) (end 161.128477 83.418075) (width 0.25) (layer "F.Cu") (net 2))
   (segment (start 136.775 88.25) (end 136.775 87.2675) (width 0.25) (layer "F.Cu") (net 2))
-  (segment (start 148.128 94.128) (end 149 95) (width 0.25) (layer "F.Cu") (net 2))
   (segment (start 134.06 90.58645) (end 135.34645 89.3) (width 0.25) (layer "F.Cu") (net 2))
   (segment (start 143.413 93.304) (end 148.128 88.589) (width 0.25) (layer "F.Cu") (net 2))
@@
   (segment (start 136.008789 92.104761) (end 136.404028 92.5) (width 0.25) (layer "F.Cu") (net 2))
   (segment (start 136.8 82.9125) (end 134.9375 81.05) (width 0.25) (layer "F.Cu") (net 2))
-  (via (at 142.5 92.5) (size 0.8) (drill 0.4) (layers "F.Cu" "B.Cu") (net 2))
   (via (at 134.5 83) (size 0.8) (drill 0.4) (layers "F.Cu" "B.Cu") (net 2))
   (via (at 161.128477 83.418075) (size 0.8) (drill 0.4) (layers "F.Cu" "B.Cu") (net 2))
   (via (at 162.930525 86.122312) (size 0.8) (drill 0.4) (layers "F.Cu" "B.Cu") (net 2))
-  (via (at 149 95) (size 0.8) (drill 0.4) (layers "F.Cu" "B.Cu") (net 2))
   (via (at 138 92.5) (size 0.8) (drill 0.4) (layers "F.Cu" "B.Cu") (net 2))
   (via (at 163.576 93.472) (size 0.8) (drill 0.4) (layers "F.Cu" "B.Cu") (net 2))
@@
   (segment (start 159.5 87.4425) (end 160.4425 87.4425) (width 0.25) (layer "B.Cu") (net 2))
   (segment (start 159.6325 87.31) (end 159.5 87.4425) (width 0.25) (layer "B.Cu") (net 2))
-  (segment (start 149 95) (end 151.35 95) (width 0.25) (layer "B.Cu") (net 2))
   (segment (start 162.258976 83.418075) (end 162.805901 83.965) (width 0.25) (layer "B.Cu") (net 2))
   (segment (start 162.930525 88.369475) (end 162.15 89.15) (width 0.25) (layer "B.Cu") (net 2))
@@
   (segment (start 155 93.5) (end 151.033 97.467) (width 0.25) (layer "F.Cu") (net 11))
   (segment (start 151.033 97.467) (end 151.033 98.599) (width 0.25) (layer "F.Cu") (net 11))
-  (via (at 155 93.5) (size 0.8) (drill 0.4) (layers "F.Cu" "B.Cu") (net 11))
   (segment (start 160.55 95.45) (end 156.95 95.45) (width 0.25) (layer "B.Cu") (net 11))
   (segment (start 156.95 95.45) (end 155 93.5) (width 0.25) (layer "B.Cu") (net 11))
