File: device/PCB/impact_v1.1/impact_v1.1.kicad_pcb (KiCad board)
At the start: 2 copper layers, 33 x 29.2 mm, 24 parts, among them U1 ESP32-WROOM-32, U2 MIC5200-3.3BM-TR, U3 ADXL375BCCZ, U4 MPU-6050

Commit message: Before Computer Reset. Backu
Other:
- board text removed: "JLCJLCJLCJLC"
Changed lines of the file:
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@@
   )
   (gr_rect (start 135.89 76.2) (end 168.8568 105.41) (layer "Edge.Cuts") (width 0.1) (fill none))
-  (gr_text "JLCJLCJLCJLC" (at 164.592 77.724) (layer "B.SilkS")
-    (effects (font (size 0.9 0.7) (thickness 0.175)) (justify mirror))
-  )
   (gr_text "Property of Amogh Kashyap" (at 151.8 104.1) (layer "B.SilkS")
     (effects (font (size 1 1) (thickness 0.15)) (justify mirror))
