File: device/PCB/impact_v1.1/impact_v1.1.kicad_sch (KiCad schematic)
At the start: 24 parts, among them J1 Conn_01x01_Male, J2 Conn_01x01_Male, U1 ESP32-WROOM-32, U2 MIC5200-3.3BM-TR, U3 ADXL375BCCZ, U4 MPU-6050

Commit message: Before Computer Reset. Backu
Other:
- company: (none) -> Amogh Kashyap
Changed lines of the file:
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@@
     (date "2022-01-30")
     (rev "Version 1.1")
+    (company "Amogh Kashyap")
+    (comment 2 "Not for Commercial or Monetary Use")
+    (comment 3 "For Use with Proprietary Software")
+    (comment 4 "Property of Amogh Kashyap")
   )
   (junction (at 165.1 53.34) (diameter 0) (color 0 0 0 0)
